Commit message: changing go0 config to match params.py
removing setting gains for gazebo_ros_control because it creates issues
with homing

File: urdf/ur5.srdf.xacro (robot description, xacro)
@@ -4,5 +4,5 @@
     <joint name="shoulder_pan_joint" value="-0.32" />
     <joint name="shoulder_lift_joint" value="-0.78" />
-    <joint name="elbow_joint" value="-2.1" />
+    <joint name="elbow_joint" value="-2.56" />
     <joint name="wrist_1_joint" value="-1.63" />
     <joint name="wrist_2_joint" value="-1.57" />
